Commit message: primer ejercicio-lidar

File: puzzlebot_sim/urdf/puzzlebot.urdf (robot description, URDF)
Before this commit: robot puzzlebot, 5 links, 4 joints
Links:
- added link base_laser; visual cylinder length=0.02 radius=0.04
Joints:
- added joint base_laser_joint: type fixed, parent base_link, child base_laser, origin xyz=0 0 0.08 rpy=0 0 0

Commit message: primer ejercicio-lidar-final

File: puzzlebot_sim/urdf/puzzlebot.urdf (robot description, URDF)
Before this commit: robot puzzlebot, 6 links, 5 joints
Links:
- removed link base_laser
- link base_link: geometry visual mesh filename=package://puzzlebot_sim/meshes/MCR2_puzzlebot_jetson_lidar_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
Joints:
- removed joint base_laser_joint
- joint caster_ball_joint: origin xyz=0.10 0 -0.03 rpy=0 0 0 -> xyz=-0.22 0 -0.055 rpy=0 0 0
