Commit message: primerejercicio3

File: week3/kinematic_model/urdf/puzzlebot.urdf (robot description, URDF)
Before this commit: robot kinematic_model, 7 links, 6 joints
Links:
- removed link chassis
Joints:
- removed joint chassis_joint
- joint base_laser_joint: parent chassis -> base_link
- joint wheel_left_joint: parent chassis -> base_link
- joint wheel_right_joint: parent chassis -> base_link
